File: panels/controls/controls.kicad_pcb (KiCad board)
At the start: 2 copper layers, 240 x 150 mm, 0 parts

Commit message: Panels: control panel v2 + SAS panel v1
Other:
- board size 240 x 150 mm -> 240 x 140 mm
- board text added: "BRAKES"
- board text added: "C417347"
- board text added: "RESET"
- board text added: "TRIM"
- board text added: "ZERO"
- board text removed: "BREAK"
- board text removed: "OFF"

Commit message: Panels: rework of ctrl and sas. Add gauges and v1 of executive
Other:
- outline, holes or cut-outs redrawn
- board text removed: "BRAKES"
- board text removed: "C111418"
- board text removed: "C1788498"
- board text removed: "C417347"
- board text removed: "EG2001-ND"
- board text removed: "LOCK"
