File: schematics/mainboard/mainboard.kicad_sch (KiCad schematic)
At the start: 82 parts, among them J1 ICSP, J10 Conn_01x02_Pin, J11 Conn_02x16_Counter_Clockwise, J2 USB_B_Micro, J3 DEALON DC-S050-200, J4 PWR_SELECT, J5 JOY1, J6 JOY2, J7 Conn_01x06_Pin, J8 DGAUGES, J9 LCD, Q2 BC849, U1 ATmega2560-16A, U2 FT232RL, U3 USBLC6-2P6, U4 AIP78M05, U5 L9110, U6 74HC595, U7 74HC595, U8 74HC165, U9 74HC165, Y1 16Mhz

Commit message: SCH:MB=> fixes + gen jlc fab prj
Parts:
- C1, C2, C3, C5: value 0.1uF -> 100nF
- C13, C14, C15, C16: value 0.1 µf -> 100nF
- J10: value Conn_01x02_Pin -> Conn_AGauge
- J11: value Conn_02x16_Counter_Clockwise -> Conn_SAS
- J5: value JOY1 -> Conn_Joy1
- J6: value JOY2 -> Conn_Joy2
- J7: value Conn_01x06_Pin -> Conn_Throttle
- J8: value DGAUGES -> Conn_DGauges
- J9: value LCD -> Conn_LCD
Connections:
- net +5V: now also C9.1, U3.5 (VBUS)
- net GND: now also C9.2, U3.2 (GND)
- net at F1.2, J4.3 (Pin_3): no longer C9.1, U3.5 (VBUS)
Other:
- note removed: "AGAUGE"
Changed lines of the file:
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@@
   (junction (at 107.315 246.38) (diameter 0) (color 0 0 0 0)
   )
+  (junction (at 408.305 203.835) (diameter 0) (color 0 0 0 0)
+  )
   (junction (at 155.575 241.3) (diameter 0) (color 0 0 0 0)
   )
@@
   (junction (at 176.53 248.92) (diameter 0) (color 0 0 0 0)
   )
+  (junction (at 398.78 172.085) (diameter 0) (color 0 0 0 0)
+  )
   (junction (at 104.775 243.84) (diameter 0) (color 0 0 0 0)
   )
@@
     (stroke (width 0) (type default))
   )
-  (wire (pts (xy 422.275 186.69) (xy 422.275 182.88))
+  (wire (pts (xy 422.275 176.53) (xy 422.275 186.69))
     (stroke (width 0) (type default))
   )
@@
     (stroke (width 0) (type default))
   )
-  (wire (pts (xy 390.525 203.2) (xy 408.305 203.2))
+  (wire (pts (xy 390.525 203.835) (xy 408.305 203.835))
     (stroke (width 0) (type default))
   )
@@
     (stroke (width 0) (type default))
   )
+  (wire (pts (xy 405.13 176.53) (xy 405.13 174.625))
+    (stroke (width 0) (type default))
+  )
   (wire (pts (xy 212.725 128.27) (xy 212.725 133.985))
     (stroke (width 0) (type default))
@@
     (stroke (width 0) (type default))
   )
+  (wire (pts (xy 422.275 176.53) (xy 405.13 176.53))
+    (stroke (width 0) (type default))
+  )
   (wire (pts (xy 400.685 301.625) (xy 400.685 298.45))
     (stroke (width 0) (type default))
@@
     (stroke (width 0) (type default))
   )
-  (wire (pts (xy 408.305 174.625) (xy 408.305 182.88))
-    (stroke (width 0) (type default))
-  )
   (wire (pts (xy 305.435 153.67) (xy 290.195 153.67))
     (stroke (width 0) (type default))
@@
     (stroke (width 0) (type default))
   )
+  (wire (pts (xy 398.78 172.085) (xy 398.78 179.705))
+    (stroke (width 0) (type default))
+  )
   (wire (pts (xy 116.84 220.98) (xy 132.715 220.98))
     (stroke (width 0) (type default))
@@
     (stroke (width 0) (type default))
   )
+  (wire (pts (xy 398.78 179.705) (xy 408.305 179.705))
+    (stroke (width 0) (type default))
+  )
   (wire (pts (xy 250.825 115.57) (xy 249.555 115.57))
     (stroke (width 0) (type default))
@@
     (stroke (width 0) (type default))
   )
+  (wire (pts (xy 405.13 174.625) (xy 408.305 174.625))
+    (stroke (width 0) (type default))
+  )
   (wire (pts (xy 449.58 203.835) (xy 447.04 203.835))
     (stroke (width 0) (type default))
@@
     (stroke (width 0) (type default))
   )
-  (wire (pts (xy 422.275 182.88) (xy 408.305 182.88))
-    (stroke (width 0) (type default))
-  )
   (bus (pts (xy 107.315 269.24) (xy 109.855 269.24))
     (stroke (width 0) (type default))
@@
     (stroke (width 0) (type default))
   )
+  (wire (pts (xy 408.305 179.705) (xy 408.305 182.88))
+    (stroke (width 0) (type default))
+  )
   (wire (pts (xy 439.42 191.77) (xy 430.53 191.77))
     (stroke (width 0) (type default))
@@
     (stroke (width 0) (type default))
   )
-  (wire (pts (xy 390.525 196.215) (xy 390.525 203.2))
+  (wire (pts (xy 390.525 196.215) (xy 390.525 203.835))
+    (stroke (width 0) (type default))
+  )
+  (wire (pts (xy 408.305 203.835) (xy 447.04 203.835))
     (stroke (width 0) (type default))
   )
@@
     (stroke (width 0) (type default))
   )
+  (wire (pts (xy 408.305 203.2) (xy 408.305 203.835))
+    (stroke (width 0) (type default))
+  )
   (wire (pts (xy 260.985 252.095) (xy 290.195 252.095))
     (stroke (width 0) (type default))
@@
     (effects (font (size 1.27 1.27)) (justify right bottom))
   )
-  (text "AGAUGE" (at 370.205 201.295 0)
-    (effects (font (size 1.27 1.27)) (justify right bottom))
-  )
   (text "ADC1" (at 274.955 222.885 0)
     (effects (font (size 1.27 1.27)) (justify left bottom))
@@
       (effects (font (size 1.27 1.27)))
     )
-    (property "Value" "Conn_02x16_Counter_Clockwise" (at 123.19 185.42 0)
+    (property "Value" "Conn_SAS" (at 123.19 185.42 0)
       (effects (font (size 1.27 1.27)) hide)
     )
@@
       (effects (font (size 1.27 1.27)) (justify left))
     )
-    (property "Value" "0.1uF" (at 321.31 106.045 0)
+    (property "Value" "100nF" (at 321.31 106.045 0)
       (effects (font (size 1.27 1.27)) (justify left))
     )
@@
   )
   (symbol (lib_id "Connector:Conn_01x02_Pin") (at 364.49 207.645 180) (unit 1)
-    (in_bom yes) (on_board yes) (dnp no) (fields_autoplaced)
-    (property "Reference" "J10" (at 366.395 205.74 0)
+    (in_bom yes) (on_board yes) (dnp no)
+    (property "Reference" "J10" (at 360.68 200.66 0)
       (effects (font (size 1.27 1.27)) (justify right))
     )
-    (property "Value" "Conn_01x02_Pin" (at 366.395 208.28 0)
+    (property "Value" "Conn_AGauge" (at 366.395 212.09 90)
       (effects (font (size 1.27 1.27)) (justify right))
     )
@@
       (effects (font (size 1.27 1.27)) (justify left))
     )
-    (property "Value" "0.1 µf" (at 176.53 159.385 0)
+    (property "Value" "100nF" (at 176.53 159.385 0)
       (effects (font (size 1.27 1.27)) (justify left))
     )
@@
       (effects (font (size 1.27 1.27)) (justify left))
     )
-    (property "Value" "0.1 µf" (at 116.84 227.33 0)
+    (property "Value" "100nF" (at 116.84 227.33 0)
       (effects (font (size 1.27 1.27)) (justify left))
     )
@@
       (effects (font (size 1.27 1.27)) (justify left))
     )
-    (property "Value" "0.1 µf" (at 183.515 227.33 0)
+    (property "Value" "100nF" (at 183.515 227.33 0)
       (effects (font (size 1.27 1.27)) (justify left))
     )
@@
       (effects (font (size 1.27 1.27)) (justify left))
     )
-    (property "Value" "0.1uF" (at 336.55 106.045 0)
+    (property "Value" "100nF" (at 336.55 106.045 0)
       (effects (font (size 1.27 1.27)) (justify left))
     )
@@
       (effects (font (size 1.27 1.27)))
     )
-    (property "Value" "Conn_01x06_Pin" (at 250.825 320.04 90)
+    (property "Value" "Conn_Throttle" (at 250.825 320.04 90)
       (effects (font (size 1.27 1.27)))
     )
@@
       (effects (font (size 1.27 1.27)) (justify left))
     )
-    (property "Value" "0.1 µf" (at 182.245 208.28 0)
+    (property "Value" "100nF" (at 182.245 208.28 0)
       (effects (font (size 1.27 1.27)) (justify left))
     )
@@
       (effects (font (size 1.27 1.27)) (justify left))
     )
-    (property "Value" "0.1uF" (at 219.71 113.665 0)
+    (property "Value" "100nF" (at 219.71 113.665 0)
       (effects (font (size 1.27 1.27)) (justify left))
     )
@@
       (effects (font (size 1.27 1.27)))
     )
-    (property "Value" "JOY1" (at 323.215 297.18 90)
+    (property "Value" "Conn_Joy1" (at 323.215 297.18 90)
       (effects (font (size 1.27 1.27)))
     )
@@
   (symbol (lib_id "Connector:Conn_01x07_Pin") (at 333.375 177.8 180) (unit 1)
     (in_bom yes) (on_board yes) (dnp no)
-    (property "Reference" "J9" (at 334.645 170.18 0)
+    (property "Reference" "J9" (at 332.74 167.64 0)
       (effects (font (size 1.27 1.27)) (justify right))
     )
-    (property "Value" "LCD" (at 335.915 179.705 90)
+    (property "Value" "Conn_LCD" (at 334.645 182.245 90)
       (effects (font (size 1.27 1.27)) (justify right))
     )
@@
       (effects (font (size 1.27 1.27)))
     )
-    (property "Value" "JOY2" (at 297.18 297.815 90)
+    (property "Value" "Conn_Joy2" (at 297.18 297.815 90)
       (effects (font (size 1.27 1.27)))
     )
@@
   (symbol (lib_id "Connector:Conn_01x06_Pin") (at 332.105 201.93 180) (unit 1)
     (in_bom yes) (on_board yes) (dnp no)
-    (property "Reference" "J8" (at 334.01 194.31 0)
+    (property "Reference" "J8" (at 331.47 191.77 0)
       (effects (font (size 1.27 1.27)))
     )
-    (property "Value" "DGAUGES" (at 334.01 201.295 90)
+    (property "Value" "Conn_DGauges" (at 334.01 198.12 90)
       (effects (font (size 1.27 1.27)))
     )
@@
       (effects (font (size 1.27 1.27)) (justify left))
     )
-    (property "Value" "0.1uF" (at 328.93 106.045 0)
+    (property "Value" "100nF" (at 328.93 106.045 0)
       (effects (font (size 1.27 1.27)) (justify left))
     )
